File: 8-BitSteck/8-BitSteck.sch (KiCad schematic (older format))
At the start: 0 parts

Commit message: Add files via upload
Connections:
- net labels added: bus0, bus1, bus2, bus3, bus4, bus5, bus6, bus7, bus[0..7]
- wire segments 0 -> 8
Changed lines of the file:
@@
 $Descr A4 11693 8268
 encoding utf-8
-Sheet 1 62
+Sheet 1 64
 Title "8-Bit FlexCPU"
 Date "2018-11-14"
 Rev "A"
 Comp "JDCoorp"
-Comment1 "Building blocks for an 8-Bit CPU"
+Comment1 ""
 Comment2 "for public use"
 Comment3 ""
-Comment4 ""
+Comment4 "Building blocks for an 8-Bit CPU"
 $EndDescr
 $Sheet
-S 7200 1300 550  450
+S 7200 1300 550  200
 U 5BD0EC1C
 F0 "clock" 50
 F1 "clock.sch" 50
-F2 "Clock" I R 7750 1550 50
+F2 "Clock" I R 7750 1400 50
 $EndSheet
 $Sheet
-S 3750 1400 550  900
+S 3750 1400 550  200
 U 5BD2AC42
 F0 "8Bit?" 50
 F1 "8Bit.sch" 50
-F2 "BIT_0(LSB)" I L 3750 1500 50
-F3 "1" I L 3750 1600 50
-F4 "2" I L 3750 1700 50
-F5 "3" I L 3750 1800 50
-F6 "4" I L 3750 1900 50
-F7 "5" I L 3750 2000 50
-F8 "6" I L 3750 2100 50
-F9 "7" I L 3750 2200 50
+F2 "BUS[0..7]" I L 3750 1500 50
 $EndSheet
 $Sheet
-S 6250 1300 500  400
+S 5850 3150 800  1450
 U 5BD2B43F
 F0 "multlogic" 50
 F1 "multlogic.sch" 50
+F2 "AND_A" I L 5850 3250 50
+F3 "AND_B" I L 5850 3350 50
+F4 "AND_C" I L 5850 3450 50
+F5 "AND_D" I L 5850 3550 50
+F6 "OR_A" I L 5850 3700 50
+F7 "OR_B" I L 5850 3800 50
+F8 "OR_C" I L 5850 3900 50
+F9 "OR_D" I L 5850 4000 50
+F10 "NAND_A" I L 5850 4150 50
+F11 "NAND_B" I L 5850 4250 50
+F12 "NOR_A" I L 5850 4400 50
+F13 "NOR_B" I L 5850 4500 50
+F14 "AND_Q" O R 6650 3400 50
+F15 "OR_Q" O R 6650 3850 50
+F16 "NAND_Q" O R 6650 4200 50
+F17 "NOR_Q" O R 6650 4450 50
 $EndSheet
 $Sheet
-S 5250 1400 550  200
+S 4650 1400 550  200
 U 5BDE2529
 F0 "1Bit?" 50
 F1 "1Bit.sch" 50
-F2 "Signal" I L 5250 1500 50
+F2 "Signal" I L 4650 1500 50
 $EndSheet
 $Sheet
-S 5250 1900 550  400
+S 4700 1900 550  200
 U 5BE1A0B6
 F0 "Sheet5BE1A0B5" 50
 F1 "8Bit_CONST.sch" 50
+F2 "OUT[0..7]" O R 5250 2000 50
 $EndSheet
 $Sheet
-S 6250 1900 500  400
+S 6250 1900 550  950
 U 5BE1C820
 F0 "Sheet5BE1C81F" 50
 F1 "1Bit_CONST.sch" 50
+F2 "HI1" O R 6800 2100 50
+F3 "HI2" O R 6800 2200 50
+F4 "HI3" O R 6800 2300 50
+F5 "HI0" O R 6800 2000 50
+F6 "LO0" O R 6800 2450 50
+F7 "LO1" O R 6800 2550 50
+F8 "LO2" O R 6800 2650 50
+F9 "LO3" O R 6800 2750 50
 $EndSheet
 $Sheet
-S 3750 2650 550  250
+S 3450 2700 800  550
 U 5BE1CDAC
 F0 "Sheet5BE1CDAB" 50
 F1 "MUX.sch" 50
+F2 "A[0..7]" I L 3450 2800 50
+F3 "B[0..7]" I L 3450 2900 50
+F4 "OUT[0..7]" O R 4250 2850 50
+F5 "S" I L 3450 3050 50
+F6 "~E" I L 3450 3150 50
 $EndSheet
 $Sheet
@@
 $EndSheet
 $Sheet
-S 2800 1400 550  900
+S 2800 1400 550  200
 U 5BE4465D
 F0 "Sheet5BE4465C" 50
 F1 "8Bit_LEDs.sch" 50
-F2 "BIT_0(LSB)" I L 2800 1500 50
-F3 "1" I L 2800 1600 50
-F4 "2" I L 2800 1700 50
-F5 "3" I L 2800 1800 50
-F6 "4" I L 2800 1900 50
-F7 "5" I L 2800 2000 50
-F8 "6" I L 2800 2100 50
-F9 "7" I L 2800 2200 50
+F2 "BUS[0..7]" I L 2800 1500 50
 $EndSheet
 $Sheet
@@
 F1 "alu.sch" 50
 $EndSheet
+Wire Bus Line
+	1850 1500 1550 1500
+Entry Wire Line
+	1450 1550 1550 1650
+Entry Wire Line
+	1450 1650 1550 1750
+Entry Wire Line
+	1450 1750 1550 1850
+Entry Wire Line
+	1450 1850 1550 1950
+Entry Wire Line
+	1450 1950 1550 2050
+Entry Wire Line
+	1450 2050 1550 2150
+Entry Wire Line
+	1450 2150 1550 2250
+Entry Wire Line
+	1450 2250 1550 2350
+Text Label 1550 1500 0    50   ~ 0
+bus[0..7]
+Wire Wire Line
+	1450 1550 1000 1550
+Wire Wire Line
+	1450 1650 1000 1650
+Wire Wire Line
+	1450 1750 1000 1750
+Wire Wire Line
+	1450 1850 1000 1850
+Wire Wire Line
+	1450 1950 1000 1950
+Wire Wire Line
+	1450 2050 1000 2050
+Wire Wire Line
+	1450 2150 1000 2150
+Wire Wire Line
+	1450 2250 1000 2250
+Text Label 1100 1550 0    50   ~ 0
+bus0
+Text Label 1100 1650 0    50   ~ 0
+bus1
+Text Label 1100 1750 0    50   ~ 0
+bus2
+Text Label 1100 1850 0    50   ~ 0
+bus3
+Text Label 1100 1950 0    50   ~ 0
+bus4
+Text Label 1100 2050 0    50   ~ 0
+bus5
+Text Label 1100 2150 0    50   ~ 0
+bus6
+Text Label 1100 2250 0    50   ~ 0
+bus7
+Wire Bus Line
+	1550 1500 1550 2350
 $EndSCHEMATC

Commit message: Multilogic routed
Connections:
- net labels removed: bus0, bus1, bus2, bus3, bus4, bus5, bus6, bus7, bus[0..7]
- wire segments 8 -> 0
Changed lines of the file:
@@
 $Descr A4 11693 8268
 encoding utf-8
-Sheet 1 64
+Sheet 1 66
 Title "8-Bit FlexCPU"
 Date "2018-11-14"
@@
 $EndSheet
 $Sheet
-S 5250 2650 550  250
+S 3400 4050 900  1050
 U 5BE42934
 F0 "Sheet5BE42933" 50
 F1 "SM.sch" 50
+F2 "IN[0..7]" I L 3400 4150 50
+F3 "OUT[0..7]" O R 4300 4150 50
+F4 "bus_0" O R 4300 4300 50
+F5 "bus_1" O R 4300 4400 50
+F6 "bus_2" O R 4300 4500 50
+F7 "bus_3" O R 4300 4600 50
+F8 "bus_4" O R 4300 4700 50
+F9 "bus_5" O R 4300 4800 50
+F10 "bus_6" O R 4300 4900 50
+F11 "bus_7" O R 4300 5000 50
 $EndSheet
 $Sheet
@@
 $EndSheet
 $Sheet
-S 7200 1900 550  300
+S 7200 1900 1000 600
 U 5BE65893
 F0 "Sheet5BE65892" 50
 F1 "alu.sch" 50
+F2 "A[0..7]" I L 7200 2000 50
+F3 "B[0..7]" I L 7200 2100 50
+F4 "S[0..3]" I L 7200 2250 50
+F5 "C_in" I L 7200 2400 50
+F6 "C_out" O R 8200 2400 50
+F7 "A=B" O R 8200 2300 50
+F8 "OUT[0..7]" O R 8200 2050 50
 $EndSheet
-Wire Bus Line
-	1850 1500 1550 1500
-Entry Wire Line
-	1450 1550 1550 1650
-Entry Wire Line
-	1450 1650 1550 1750
-Entry Wire Line
-	1450 1750 1550 1850
-Entry Wire Line
-	1450 1850 1550 1950
-Entry Wire Line
-	1450 1950 1550 2050
-Entry Wire Line
-	1450 2050 1550 2150
-Entry Wire Line
-	1450 2150 1550 2250
-Entry Wire Line
-	1450 2250 1550 2350
-Text Label 1550 1500 0    50   ~ 0
-bus[0..7]
-Wire Wire Line
-	1450 1550 1000 1550
-Wire Wire Line
-	1450 1650 1000 1650
-Wire Wire Line
-	1450 1750 1000 1750
-Wire Wire Line
-	1450 1850 1000 1850
-Wire Wire Line
-	1450 1950 1000 1950
-Wire Wire Line
-	1450 2050 1000 2050
-Wire Wire Line
-	1450 2150 1000 2150
-Wire Wire Line
-	1450 2250 1000 2250
-Text Label 1100 1550 0    50   ~ 0
-bus0
-Text Label 1100 1650 0    50   ~ 0
-bus1
-Text Label 1100 1750 0    50   ~ 0
-bus2
-Text Label 1100 1850 0    50   ~ 0
-bus3
-Text Label 1100 1950 0    50   ~ 0
-bus4
-Text Label 1100 2050 0    50   ~ 0
-bus5
-Text Label 1100 2150 0    50   ~ 0
-bus6
-Text Label 1100 2250 0    50   ~ 0
-bus7
-Wire Bus Line
-	1550 1500 1550 2350
 $EndSCHEMATC
