File: 8-BitSteck/alu.sch (KiCad schematic (older format))
At the start: 4 parts

Commit message: Multilogic routed
Connections:
- net labels added: A=B, A[0..7], B[0..7], C_in, C_out, OUT[0..7], S[0..3], a0, a1, a2, a3, a4, a5, a6, a7, a[0..7], b0, b1, b2, b3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
- net labels removed: A_0, A_1, A_2, A_3, A_4, A_5, A_6, A_7, B_0, B_1, B_2, B_3, B_4, B_5, B_6, B_7
- wire segments 114 -> 71
