File: 8-BitSteck/clock.sch (KiCad schematic (older format))
At the start: 7 parts, among them U1 NE555

Commit message: Multilogic routed
Parts:
- removed D1: LED_BLUE, LED_SMD:LED_0603_1608Metric_Pad1.05x0.95mm_HandSolder, symbol Device:LED
- removed R2: 80, Resistor_SMD:R_0603_1608Metric_Pad1.05x0.95mm_HandSolder, symbol Device:R
- renumbered C2 to C1, C1 to C2
Connections:
- wire segments 34 -> 29
Changed lines of the file:
@@
 EESchema Schematic File Version 4
-LIBS:8-BitSteck-cache
 EELAYER 26 0
 EELAYER END
 $Descr A4 11693 8268
 encoding utf-8
-Sheet 2 64
+Sheet 1 2
 Title ""
 Date ""
@@
 $EndComp
 $Comp
-L power:+3.3V #PWR0101
+L power:+3.3V #PWR01
 U 1 1 5BD0ED0B
 P 3050 2550
-F 0 "#PWR0101" H 3050 2400 50  0001 C CNN
+F 0 "#PWR01" H 3050 2400 50  0001 C CNN
 F 1 "+3.3V" H 3065 2723 50  0000 C CNN
 F 2 "" H 3050 2550 50  0001 C CNN
@@
 $EndComp
 $Comp
-L power:GND #PWR0102
+L power:GND #PWR02
 U 1 1 5BD0ED67
 P 3050 4100
-F 0 "#PWR0102" H 3050 3850 50  0001 C CNN
+F 0 "#PWR02" H 3050 3850 50  0001 C CNN
 F 1 "GND" H 3055 3927 50  0000 C CNN
 F 2 "" H 3050 4100 50  0001 C CNN
@@
 	3550 3600 3550 3350
 $Comp
-L Device:C C1
+L Device:C C2
 U 1 1 5BD0EE42
 P 3550 3750
-F 0 "C1" H 3665 3796 50  0000 L CNN
+F 0 "C2" H 3665 3796 50  0000 L CNN
 F 1 "0.01uF" H 3665 3705 50  0000 L CNN
 F 2 "Capacitor_SMD:C_0603_1608Metric_Pad1.05x0.95mm_HandSolder" H 3588 3600 50  0001 C CNN
@@
 	3050 3900 3050 3550
 $Comp
-L Device:C C2
+L Device:C C1
 U 1 1 5BD0F054
 P 2450 3850
-F 0 "C2" H 2565 3896 50  0000 L CNN
+F 0 "C1" H 2565 3896 50  0000 L CNN
 F 1 "0.01uF" H 2565 3805 50  0000 L CNN
 F 2 "Capacitor_SMD:C_0603_1608Metric_Pad1.05x0.95mm_HandSolder" H 2488 3700 50  0001 C CNN
@@
 Wire Wire Line
 	3650 2450 3700 2450
+Connection ~ 3650 2650
+Wire Wire Line
+	3650 2650 3650 2450
+Wire Wire Line
+	3050 3900 3550 3900
 $Sheet
 S 4950 2450 550  400
@@
 F2 "Signal" I L 4950 2650 50
 $EndSheet
-Connection ~ 3650 2650
 Wire Wire Line
-	3650 2650 3650 2450
-Wire Wire Line
-	3650 2650 4450 2650
-$Comp
-L Device:LED D1
-U 1 1 5BD291EE
-P 4450 3250
-F 0 "D1" V 4488 3133 50  0000 R CNN
-F 1 "LED_BLUE" V 4397 3133 50  0000 R CNN
-F 2 "LED_SMD:LED_0603_1608Metric_Pad1.05x0.95mm_HandSolder" H 4450 3250 50  0001 C CNN
-F 3 "~" H 4450 3250 50  0001 C CNN
-	1    4450 3250
-	0    -1   -1   0
-$EndComp
-$Comp
-L Device:R R2
-U 1 1 5BD29AE4
-P 4450 2900
-F 0 "R2" H 4520 2946 50  0000 L CNN
-F 1 "80" H 4520 2855 50  0000 L CNN
-F 2 "Resistor_SMD:R_0603_1608Metric_Pad1.05x0.95mm_HandSolder" V 4380 2900 50  0001 C CNN
-F 3 "~" H 4450 2900 50  0001 C CNN
-	1    4450 2900
-	1    0    0    -1
-$EndComp
-Wire Wire Line
-	4450 2650 4450 2750
-Connection ~ 4450 2650
-Wire Wire Line
-	4450 2650 4950 2650
-Wire Wire Line
-	4450 3050 4450 3100
-Wire Wire Line
-	3050 3900 3550 3900
-Connection ~ 3550 3900
-Wire Wire Line
-	3550 3900 4450 3900
-Wire Wire Line
-	4450 3400 4450 3900
+	3650 2650 4950 2650
 $EndSCHEMATC
