File: 8-BitSteck/multlogic.sch (KiCad schematic (older format))
At the start: 22 parts

Commit message: Add files via upload
Connections:
- net labels added: AND_A, AND_B, AND_C, AND_D, AND_Q, NAND_A, NAND_B, NAND_Q, NOR_A, NOR_B, NOR_Q, OR_A, OR_B, OR_C, OR_D, OR_Q
- wire segments 88 -> 136
Other:
- moved on the sheet: U?E

Commit message: Multilogic routed
Parts:
- removed R? (x12): R_default, symbol Device:R
- added R1, R2, R3, R4: R, Resistor_SMD:R_0603_1608Metric_Pad1.05x0.95mm_HandSolder, symbol Device:R
- added RN2, RN3: R_Pack04, Resistor_SMD:R_Array_Convex_4x0603, symbol Device:R_Pack04
- U1, U2: renamed from U?; footprint (none) -> Package_SO:SOIC-14_3.9x8.7mm_P1.27mm
Connections:
- net labels added: R_Pullup1, R_Pullup2
- wire segments 136 -> 170
Other:
- moved on the sheet: U1B, U1C, U1D, U1E, U2B, U2C, U2D, U2E
