File: 8-BitSteck/1Bit.sch (KiCad schematic (older format))
At the start: 4 parts

Commit message: Multilogic routed
Parts:
- D1: renamed from D?; footprint (none) -> LED_SMD:LED_0603_1608Metric_Pad1.05x0.95mm_HandSolder
- R13: renamed from R?; footprint (none) -> Resistor_SMD:R_0603_1608Metric_Pad1.05x0.95mm_HandSolder
- gave numbers to parts that had none: 2

Commit message: 8-bit-Const routed
Parts:
- renumbered R13 to R3
