File: 8-BitSteck/8Bit_CONST.sch (KiCad schematic (older format))
At the start: 9 parts

Commit message: Add files via upload
Connections:
- net labels added: OUT[0..7], bus0, bus1, bus2, bus3, bus4, bus5, bus6, bus7, bus[0..7]
Changed lines of the file:
@@
 $Descr A4 11693 8268
 encoding utf-8
-Sheet 23 62
+Sheet 23 64
 Title ""
 Date ""
@@
 Comment4 ""
 $EndDescr
-$Sheet
-S 5550 2450 550  900
-U 5BE1A194
-F0 "sheet5BE1A18A" 50
-F1 "8Bit.sch" 50
-F2 "BIT_0(LSB)" I L 5550 2550 50
-F3 "1" I L 5550 2650 50
-F4 "2" I L 5550 2750 50
-F5 "3" I L 5550 2850 50
-F6 "4" I L 5550 2950 50
-F7 "5" I L 5550 3050 50
-F8 "6" I L 5550 3150 50
-F9 "7" I L 5550 3250 50
-$EndSheet
 $Comp
 L Switch:SW_DIP_x08 SW?
@@
 Wire Wire Line
 	4100 2300 4100 2550
+Wire Wire Line
+	4250 2300 4250 2650
+Wire Wire Line
+	4400 2300 4400 2750
+Wire Wire Line
+	4550 2300 4550 2850
+Wire Wire Line
+	4700 2300 4700 2950
+Wire Wire Line
+	4850 2300 4850 3050
+Wire Wire Line
+	5000 2300 5000 3150
+Wire Wire Line
+	5150 2300 5150 3250
+Entry Wire Line
+	5850 2550 5950 2650
+Entry Wire Line
+	5850 2650 5950 2750
+Entry Wire Line
+	5850 2750 5950 2850
+Entry Wire Line
+	5850 2850 5950 2950
+Entry Wire Line
+	5850 2950 5950 3050
+Entry Wire Line
+	5850 3050 5950 3150
+Entry Wire Line
+	5850 3150 5950 3250
+Entry Wire Line
+	5850 3250 5950 3350
+Text Label 6050 2100 0    50   ~ 0
+bus[0..7]
+Text Label 5500 2550 0    50   ~ 0
+bus0
+Text Label 5500 2650 0    50   ~ 0
+bus1
+Text Label 5500 2750 0    50   ~ 0
+bus2
+Text Label 5500 2850 0    50   ~ 0
+bus3
+Text Label 5500 2950 0    50   ~ 0
+bus4
+Text Label 5500 3050 0    50   ~ 0
+bus5
+Text Label 5500 3150 0    50   ~ 0
+bus6
+Text Label 5500 3250 0    50   ~ 0
+bus7
+Wire Wire Line
+	4100 2550 5850 2550
 Connection ~ 4100 2550
 Wire Wire Line
-	4250 2300 4250 2650
+	4250 2650 5850 2650
 Connection ~ 4250 2650
 Wire Wire Line
-	4400 2300 4400 2750
+	4400 2750 5850 2750
 Connection ~ 4400 2750
 Wire Wire Line
-	4550 2300 4550 2850
+	4550 2850 5850 2850
 Connection ~ 4550 2850
 Wire Wire Line
-	4700 2300 4700 2950
+	4700 2950 5850 2950
 Connection ~ 4700 2950
 Wire Wire Line
-	4850 2300 4850 3050
+	4850 3050 5850 3050
 Connection ~ 4850 3050
 Wire Wire Line
-	5000 2300 5000 3150
+	5000 3150 5850 3150
 Connection ~ 5000 3150
 Wire Wire Line
-	5150 2300 5150 3250
+	5150 3250 5850 3250
 Connection ~ 5150 3250
 $Sheet
-S 6450 2450 550  900
-U 5BE6278D
-F0 "sheet5BE62783" 50
+S 6500 2000 550  200
+U 5BF47295
+F0 "sheet5BF47291" 50
+F1 "8Bit.sch" 50
+F2 "BUS[0..8]" I L 6500 2100 50
+$EndSheet
+$Sheet
+S 6500 2400 550  200
+U 5BF47298
+F0 "sheet5BF47292" 50
 F1 "8Bit_LEDs.sch" 50
-F2 "BIT_0(LSB)" I L 6450 2550 50
-F3 "1" I L 6450 2650 50
-F4 "2" I L 6450 2750 50
-F5 "3" I L 6450 2850 50
-F6 "4" I L 6450 2950 50
-F7 "5" I L 6450 3050 50
-F8 "6" I L 6450 3150 50
-F9 "7" I L 6450 3250 50
+F2 "BUS[0..8]" I L 6500 2500 50
 $EndSheet
-Wire Wire Line
-	4100 2550 6450 2550
-Wire Wire Line
-	4250 2650 6450 2650
-Wire Wire Line
-	4400 2750 6450 2750
-Wire Wire Line
-	4550 2850 6450 2850
-Wire Wire Line
-	4700 2950 6450 2950
-Wire Wire Line
-	4850 3050 6450 3050
-Wire Wire Line
-	5000 3150 6450 3150
-Wire Wire Line
-	5150 3250 6450 3250
+Wire Bus Line
+	6500 2100 5950 2100
+Wire Bus Line
+	5950 2100 5950 2500
+Connection ~ 5950 2500
+Wire Bus Line
+	5950 2500 6500 2500
+Text HLabel 6500 2950 2    50   Output ~ 0
+OUT[0..7]
+Wire Bus Line
+	6500 2950 5950 2950
+Connection ~ 5950 2950
+Wire Bus Line
+	5950 2500 5950 2950
+Wire Bus Line
+	5950 2950 5950 3350
 $EndSCHEMATC

Commit message: 8-bit-Const routed
Parts:
- removed R? (x8): R_CONST, symbol Device:R
- added RN1, RN2: R_Pack04, Resistor_SMD:R_Array_Convex_4x0603, symbol Device:R_Pack04
- SW1: renamed from SW?; footprint (none) -> Button_Switch_SMD:SW_DIP_SPSTx08_Slide_6.7x21.88mm_W8.61mm_P2.54mm_LowProfile
Connections:
- wire segments 39 -> 49
Changed lines of the file:
@@
 EESchema Schematic File Version 4
-LIBS:8-BitSteck-cache
 EELAYER 26 0
 EELAYER END
 $Descr A4 11693 8268
 encoding utf-8
-Sheet 23 66
+Sheet 1 3
 Title ""
 Date ""
@@
 $EndDescr
 $Comp
-L Switch:SW_DIP_x08 SW?
+L Switch:SW_DIP_x08 SW1
 U 1 1 5BE1A1C6
 P 3800 2950
-F 0 "SW?" H 3800 3617 50  0000 C CNN
+F 0 "SW1" H 3800 3617 50  0000 C CNN
 F 1 "SW_DIP_x08" H 3800 3526 50  0000 C CNN
-F 2 "" H 3800 2950 50  0001 C CNN
+F 2 "Button_Switch_SMD:SW_DIP_SPSTx08_Slide_6.7x21.88mm_W8.61mm_P2.54mm_LowProfile" H 3800 2950 50  0001 C CNN
 F 3 "" H 3800 2950 50  0001 C CNN
 	1    3800 2950
@@
 $EndComp
 $Comp
-L power:GND #PWR?
+L power:GND #PWR01
 U 1 1 5BE1A278
 P 3500 3450
-F 0 "#PWR?" H 3500 3200 50  0001 C CNN
+F 0 "#PWR01" H 3500 3200 50  0001 C CNN
 F 1 "GND" H 3505 3277 50  0000 C CNN
 F 2 "" H 3500 3450 50  0001 C CNN
@@
 	4100 3250 5150 3250
 $Comp
-L Device:R R?
-U 1 1 5BE1A5E9
-P 4100 2150
-F 0 "R?" H 4170 2196 50  0000 L CNN
-F 1 "R_CONST" H 4170 2105 50  0000 L CNN
-F 2 "" V 4030 2150 50  0001 C CNN
-F 3 "~" H 4100 2150 50  0001 C CNN
-	1    4100 2150
-	1    0    0    -1
-$EndComp
-$Comp
-L Device:R R?
-U 1 1 5BE1A722
-P 4250 2150
-F 0 "R?" H 4320 2196 50  0000 L CNN
-F 1 "R_CONST" H 4320 2105 50  0000 L CNN
-F 2 "" V 4180 2150 50  0001 C CNN
-F 3 "~" H 4250 2150 50  0001 C CNN
-	1    4250 2150
-	1    0    0    -1
-$EndComp
-$Comp
-L Device:R R?
-U 1 1 5BE1A7C9
-P 4400 2150
-F 0 "R?" H 4470 2196 50  0000 L CNN
-F 1 "R_CONST" H 4470 2105 50  0000 L CNN
-F 2 "" V 4330 2150 50  0001 C CNN
-F 3 "~" H 4400 2150 50  0001 C CNN
-	1    4400 2150
-	1    0    0    -1
-$EndComp
-$Comp
-L Device:R R?
-U 1 1 5BE1A86F
-P 4550 2150
-F 0 "R?" H 4620 2196 50  0000 L CNN
-F 1 "R_CONST" H 4620 2105 50  0000 L CNN
-F 2 "" V 4480 2150 50  0001 C CNN
-F 3 "~" H 4550 2150 50  0001 C CNN
-	1    4550 2150
-	1    0    0    -1
-$EndComp
-$Comp
-L Device:R R?
-U 1 1 5BE1A916
-P 4700 2150
-F 0 "R?" H 4770 2196 50  0000 L CNN
-F 1 "R_CONST" H 4770 2105 50  0000 L CNN
-F 2 "" V 4630 2150 50  0001 C CNN
-F 3 "~" H 4700 2150 50  0001 C CNN
-	1    4700 2150
-	1    0    0    -1
-$EndComp
-$Comp
-L Device:R R?
-U 1 1 5BE1A9BE
-P 4850 2150
-F 0 "R?" H 4920 2196 50  0000 L CNN
-F 1 "R_CONST" H 4920 2105 50  0000 L CNN
-F 2 "" V 4780 2150 50  0001 C CNN
-F 3 "~" H 4850 2150 50  0001 C CNN
-	1    4850 2150
-	1    0    0    -1
-$EndComp
-$Comp
-L Device:R R?
-U 1 1 5BE1AA67
-P 5000 2150
-F 0 "R?" H 5070 2196 50  0000 L CNN
-F 1 "R_CONST" H 5070 2105 50  0000 L CNN
-F 2 "" V 4930 2150 50  0001 C CNN
-F 3 "~" H 5000 2150 50  0001 C CNN
-	1    5000 2150
-	1    0    0    -1
-$EndComp
-$Comp
-L Device:R R?
-U 1 1 5BE1AB1B
-P 5150 2150
-F 0 "R?" H 5220 2196 50  0000 L CNN
-F 1 "R_CONST" H 5220 2105 50  0000 L CNN
-F 2 "" V 5080 2150 50  0001 C CNN
-F 3 "~" H 5150 2150 50  0001 C CNN
-	1    5150 2150
-	1    0    0    -1
-$EndComp
-$Comp
-L power:+3.3V #PWR?
+L power:+3.3V #PWR02
 U 1 1 5BE1ABD5
-P 4100 1900
-F 0 "#PWR?" H 4100 1750 50  0001 C CNN
-F 1 "+3.3V" H 4115 2073 50  0000 C CNN
-F 2 "" H 4100 1900 50  0001 C CNN
-F 3 "" H 4100 1900 50  0001 C CNN
-	1    4100 1900
-	1    0    0    -1
-$EndComp
-Wire Wire Line
-	4100 1900 4100 2000
-Wire Wire Line
-	4100 2000 4250 2000
-Connection ~ 4100 2000
-Connection ~ 4250 2000
-Wire Wire Line
-	4250 2000 4400 2000
-Connection ~ 4400 2000
-Wire Wire Line
-	4400 2000 4550 2000
-Connection ~ 4550 2000
-Wire Wire Line
-	4550 2000 4700 2000
-Connection ~ 4700 2000
-Wire Wire Line
-	4700 2000 4850 2000
-Connection ~ 4850 2000
-Wire Wire Line
-	4850 2000 5000 2000
-Connection ~ 5000 2000
-Wire Wire Line
-	5000 2000 5150 2000
-Wire Wire Line
-	4100 2300 4100 2550
+P 4200 1550
+F 0 "#PWR02" H 4200 1400 50  0001 C CNN
+F 1 "+3.3V" H 4215 1723 50  0000 C CNN
+F 2 "" H 4200 1550 50  0001 C CNN
+F 3 "" H 4200 1550 50  0001 C CNN
+	1    4200 1550
+	1    0    0    -1
+$EndComp
 Wire Wire Line
 	4250 2300 4250 2650
 Wire Wire Line
-	4400 2300 4400 2750
-Wire Wire Line
 	4550 2300 4550 2850
 Wire Wire Line
 	4700 2300 4700 2950
 Wire Wire Line
-	4850 2300 4850 3050
-Wire Wire Line
 	5000 2300 5000 3150
-Wire Wire Line
-	5150 2300 5150 3250
 Entry Wire Line
 	5850 2550 5950 2650
@@
 	6500 2950 5950 2950
 Connection ~ 5950 2950
+$Comp
+L Device:R_Pack04 RN1
+U 1 1 5BEEE138
+P 4400 2000
+F 0 "RN1" H 4588 2046 50  0000 L CNN
+F 1 "R_Pack04" H 4588 1955 50  0000 L CNN
+F 2 "Resistor_SMD:R_Array_Convex_4x0603" V 4675 2000 50  0001 C CNN
+F 3 "~" H 4400 2000 50  0001 C CNN
+	1    4400 2000
+	1    0    0    -1
+$EndComp
+$Comp
+L Device:R_Pack04 RN2
+U 1 1 5BEEE17C
+P 4950 2000
+F 0 "RN2" H 5138 2046 50  0000 L CNN
+F 1 "R_Pack04" H 5138 1955 50  0000 L CNN
+F 2 "Resistor_SMD:R_Array_Convex_4x0603" V 5225 2000 50  0001 C CNN
+F 3 "~" H 4950 2000 50  0001 C CNN
+	1    4950 2000
+	1    0    0    -1
+$EndComp
+Wire Wire Line
+	4200 1550 4200 1800
+Wire Wire Line
+	4200 1800 4300 1800
+Connection ~ 4200 1800
+Connection ~ 4300 1800
+Wire Wire Line
+	4300 1800 4400 1800
+Connection ~ 4400 1800
+Wire Wire Line
+	4400 1800 4500 1800
+Connection ~ 4500 1800
+Wire Wire Line
+	4500 1800 4750 1800
+Connection ~ 4750 1800
+Wire Wire Line
+	4750 1800 4850 1800
+Connection ~ 4850 1800
+Wire Wire Line
+	4850 1800 4950 1800
+Connection ~ 4950 1800
+Wire Wire Line
+	4950 1800 5050 1800
+Wire Wire Line
+	5050 2200 5150 2200
+Wire Wire Line
+	5150 2200 5150 3250
+Wire Wire Line
+	4950 2200 4950 2300
+Wire Wire Line
+	4950 2300 5000 2300
+Wire Wire Line
+	4850 2200 4850 3050
+Wire Wire Line
+	4750 2200 4750 2300
+Wire Wire Line
+	4750 2300 4700 2300
+Wire Wire Line
+	4550 2300 4500 2300
+Wire Wire Line
+	4500 2300 4500 2200
+Wire Wire Line
+	4400 2200 4400 2750
+Wire Wire Line
+	4250 2300 4300 2300
+Wire Wire Line
+	4300 2300 4300 2200
+Wire Wire Line
+	4200 2200 4100 2200
+Wire Wire Line
+	4100 2200 4100 2550
 Wire Bus Line
 	5950 2500 5950 2950
