File: 8-BitSteck/8Bit_LEDs.sch (KiCad schematic (older format))
At the start: 11 parts

Commit message: Add files via upload
Connections:
- net labels added: BUS[0..7], in0, in1, in2, in3, in4, in5, in6, in7, in[0..7]
- net labels removed: 1, 2, 3, 4, 5, 6, 7, BIT_0(LSB)

Commit message: Multilogic routed
Parts:
- removed RN? (x2): R_Network04, Resistor_THT:R_Array_SIP5, symbol Device:R_Network04
- added RN1, RN2: R_Pack04, Resistor_SMD:R_Array_Concave_4x0603, symbol Device:R_Pack04
- D10, D11, D12, D13, D14, D15, D16, D9: renamed from D?; footprint (none) -> LED_SMD:LED_0603_1608Metric_Pad1.05x0.95mm_HandSolder
- U1: renamed from U?; footprint (none) -> Package_SO:SOP-18_7.0x12.5mm_P1.27mm
Connections:
- wire segments 30 -> 36
Changed lines of the file:
@@
 EESchema Schematic File Version 4
-LIBS:8-BitSteck-cache
 EELAYER 26 0
 EELAYER END
 $Descr A4 11693 8268
 encoding utf-8
-Sheet 55 64
+Sheet 11 12
 Title ""
 Date ""
@@
 AR Path="/5BE1CDAC/5BF7F814/5BE44C99" Ref="U?"  Part="1"
 AR Path="/5BE1CDAC/5BF87C71/5BE44C99" Ref="U?"  Part="1"
-F 0 "U?" H 3500 4317 50  0000 C CNN
+AR Path="/5BEDDDBB/5BE44C99" Ref="U1"  Part="1"
+F 0 "U1" H 3500 4317 50  0000 C CNN
 F 1 "ULN2803A" H 3500 4226 50  0000 C CNN
-F 2 "" H 3550 3100 50  0001 L CNN
+F 2 "Package_SO:SOP-18_7.0x12.5mm_P1.27mm" H 3550 3100 50  0001 L CNN
 F 3 "http://www.ti.com/lit/ds/symlink/uln2803a.pdf" H 3600 3550 50  0001 C CNN
 	1    3500 3750
@@
 $EndComp
 $Comp
-L power:GND #PWR?
+L power:GND #PWR035
 U 1 1 5BE4524F
 P 3500 4550
-F 0 "#PWR?" H 3500 4300 50  0001 C CNN
+F 0 "#PWR035" H 3500 4300 50  0001 C CNN
 F 1 "GND" H 3505 4377 50  0000 C CNN
 F 2 "" H 3500 4550 50  0001 C CNN
@@
 $EndComp
 $Comp
-L power:+3.3V #PWR?
+L power:+3.3V #PWR036
 U 1 1 5BE4527A
 P 3950 3350
-F 0 "#PWR?" H 3950 3200 50  0001 C CNN
+F 0 "#PWR036" H 3950 3200 50  0001 C CNN
 F 1 "+3.3V" H 3965 3523 50  0000 C CNN
 F 2 "" H 3950 3350 50  0001 C CNN
@@
 Wire Wire Line
 	3950 3450 3900 3450
-$Comp
-L Device:R_Network04 RN?
-U 1 1 5BE45329
-P 5000 3750
-AR Path="/5BE4465D/5BE45329" Ref="RN?"  Part="1"
-AR Path="/5BE1A0B6/5BE6278D/5BE45329" Ref="RN?"  Part="1"
-AR Path="/5BE1CDAC/5BE47CF1/5BE45329" Ref="RN?"  Part="1"
-AR Path="/5BE42934/5BE5F20D/5BE45329" Ref="RN?"  Part="1"
-AR Path="/5BE65893/5BE65A53/5BE45329" Ref="RN?"  Part="1"
-AR Path="/5BE1A0B6/5BF47298/5BE45329" Ref="RN?"  Part="1"
-AR Path="/5BE1CDAC/5BF6FAD3/5BE45329" Ref="RN?"  Part="1"
-AR Path="/5BE1CDAC/5BF7F814/5BE45329" Ref="RN?"  Part="1"
-AR Path="/5BE1CDAC/5BF87C71/5BE45329" Ref="RN?"  Part="1"
-F 0 "RN?" V 4583 3750 50  0000 C CNN
-F 1 "R_Network04" V 4674 3750 50  0000 C CNN
-F 2 "Resistor_THT:R_Array_SIP5" V 5275 3750 50  0001 C CNN
-F 3 "http://www.vishay.com/docs/31509/csc.pdf" H 5000 3750 50  0001 C CNN
-	1    5000 3750
-	0    1    1    0
-$EndComp
-$Comp
-L Device:R_Network04 RN?
-U 1 1 5BE453B0
-P 5000 4150
-AR Path="/5BE4465D/5BE453B0" Ref="RN?"  Part="1"
-AR Path="/5BE1A0B6/5BE6278D/5BE453B0" Ref="RN?"  Part="1"
-AR Path="/5BE1CDAC/5BE47CF1/5BE453B0" Ref="RN?"  Part="1"
-AR Path="/5BE42934/5BE5F20D/5BE453B0" Ref="RN?"  Part="1"
-AR Path="/5BE65893/5BE65A53/5BE453B0" Ref="RN?"  Part="1"
-AR Path="/5BE1A0B6/5BF47298/5BE453B0" Ref="RN?"  Part="1"
-AR Path="/5BE1CDAC/5BF6FAD3/5BE453B0" Ref="RN?"  Part="1"
-AR Path="/5BE1CDAC/5BF7F814/5BE453B0" Ref="RN?"  Part="1"
-AR Path="/5BE1CDAC/5BF87C71/5BE453B0" Ref="RN?"  Part="1"
-F 0 "RN?" V 4583 4150 50  0000 C CNN
-F 1 "R_Network04" V 4674 4150 50  0000 C CNN
-F 2 "Resistor_THT:R_Array_SIP5" V 5275 4150 50  0001 C CNN
-F 3 "http://www.vishay.com/docs/31509/csc.pdf" H 5000 4150 50  0001 C CNN
-	1    5000 4150
-	0    1    1    0
-$EndComp
 Wire Wire Line
 	3500 4450 3500 4550
-Wire Wire Line
-	5200 3550 5200 3950
-Wire Wire Line
-	5200 3950 5200 4450
-Connection ~ 5200 3950
 Connection ~ 3500 4450
 $Comp
@@
 AR Path="/5BE1CDAC/5BF7F814/5BE455EA" Ref="D?"  Part="1"
 AR Path="/5BE1CDAC/5BF87C71/5BE455EA" Ref="D?"  Part="1"
-F 0 "D?" H 4492 3295 50  0000 C CNN
+AR Path="/5BEDDDBB/5BE455EA" Ref="D13"  Part="1"
+F 0 "D13" H 4492 3295 50  0000 C CNN
 F 1 "LED" H 4492 3386 50  0000 C CNN
-F 2 "" H 4500 3550 50  0001 C CNN
+F 2 "LED_SMD:LED_0603_1608Metric_Pad1.05x0.95mm_HandSolder" H 4500 3550 50  0001 C CNN
 F 3 "~" H 4500 3550 50  0001 C CNN
 	1    4500 3550
@@
 AR Path="/5BE1CDAC/5BF7F814/5BE45642" Ref="D?"  Part="1"
 AR Path="/5BE1CDAC/5BF87C71/5BE45642" Ref="D?"  Part="1"
-F 0 "D?" H 4142 3395 50  0000 C CNN
+AR Path="/5BEDDDBB/5BE45642" Ref="D9"  Part="1"
+F 0 "D9" H 4142 3395 50  0000 C CNN
 F 1 "LED" H 4142 3486 50  0000 C CNN
-F 2 "" H 4150 3650 50  0001 C CNN
+F 2 "LED_SMD:LED_0603_1608Metric_Pad1.05x0.95mm_HandSolder" H 4150 3650 50  0001 C CNN
 F 3 "~" H 4150 3650 50  0001 C CNN
 	1    4150 3650
@@
 AR Path="/5BE1CDAC/5BF7F814/5BE45666" Ref="D?"  Part="1"
 AR Path="/5BE1CDAC/5BF87C71/5BE45666" Ref="D?"  Part="1"
-F 0 "D?" H 4492 3495 50  0000 C CNN
+AR Path="/5BEDDDBB/5BE45666" Ref="D14"  Part="1"
+F 0 "D14" H 4492 3495 50  0000 C CNN
 F 1 "LED" H 4492 3586 50  0000 C CNN
-F 2 "" H 4500 3750 50  0001 C CNN
+F 2 "LED_SMD:LED_0603_1608Metric_Pad1.05x0.95mm_HandSolder" H 4500 3750 50  0001 C CNN
 F 3 "~" H 4500 3750 50  0001 C CNN
 	1    4500 3750
@@
 AR Path="/5BE1CDAC/5BF7F814/5BE45682" Ref="D?"  Part="1"
 AR Path="/5BE1CDAC/5BF87C71/5BE45682" Ref="D?"  Part="1"
-F 0 "D?" H 4142 3595 50  0000 C CNN
+AR Path="/5BEDDDBB/5BE45682" Ref="D10"  Part="1"
+F 0 "D10" H 4142 3595 50  0000 C CNN
 F 1 "LED" H 4142 3686 50  0000 C CNN
-F 2 "" H 4150 3850 50  0001 C CNN
+F 2 "LED_SMD:LED_0603_1608Metric_Pad1.05x0.95mm_HandSolder" H 4150 3850 50  0001 C CNN
 F 3 "~" H 4150 3850 50  0001 C CNN
 	1    4150 3850
@@
 AR Path="/5BE1CDAC/5BF7F814/5BE456A0" Ref="D?"  Part="1"
 AR Path="/5BE1CDAC/5BF87C71/5BE456A0" Ref="D?"  Part="1"
-F 0 "D?" H 4492 3695 50  0000 C CNN
+AR Path="/5BEDDDBB/5BE456A0" Ref="D15"  Part="1"
+F 0 "D15" H 4492 3695 50  0000 C CNN
 F 1 "LED" H 4492 3786 50  0000 C CNN
-F 2 "" H 4500 3950 50  0001 C CNN
+F 2 "LED_SMD:LED_0603_1608Metric_Pad1.05x0.95mm_HandSolder" H 4500 3950 50  0001 C CNN
 F 3 "~" H 4500 3950 50  0001 C CNN
 	1    4500 3950
@@
 AR Path="/5BE1CDAC/5BF7F814/5BE456C0" Ref="D?"  Part="1"
 AR Path="/5BE1CDAC/5BF87C71/5BE456C0" Ref="D?"  Part="1"
-F 0 "D?" H 4142 3795 50  0000 C CNN
+AR Path="/5BEDDDBB/5BE456C0" Ref="D11"  Part="1"
+F 0 "D11" H 4142 3795 50  0000 C CNN
 F 1 "LED" H 4142 3886 50  0000 C CNN
-F 2 "" H 4150 4050 50  0001 C CNN
+F 2 "LED_SMD:LED_0603_1608Metric_Pad1.05x0.95mm_HandSolder" H 4150 4050 50  0001 C CNN
 F 3 "~" H 4150 4050 50  0001 C CNN
 	1    4150 4050
@@
 AR Path="/5BE1CDAC/5BF7F814/5BE456E2" Ref="D?"  Part="1"
 AR Path="/5BE1CDAC/5BF87C71/5BE456E2" Ref="D?"  Part="1"
-F 0 "D?" H 4492 3895 50  0000 C CNN
+AR Path="/5BEDDDBB/5BE456E2" Ref="D16"  Part="1"
+F 0 "D16" H 4492 3895 50  0000 C CNN
 F 1 "LED" H 4492 3986 50  0000 C CNN
-F 2 "" H 4500 4150 50  0001 C CNN
+F 2 "LED_SMD:LED_0603_1608Metric_Pad1.05x0.95mm_HandSolder" H 4500 4150 50  0001 C CNN
 F 3 "~" H 4500 4150 50  0001 C CNN
 	1    4500 4150
@@
 AR Path="/5BE1CDAC/5BF7F814/5BE45706" Ref="D?"  Part="1"
 AR Path="/5BE1CDAC/5BF87C71/5BE45706" Ref="D?"  Part="1"
-F 0 "D?" H 4142 3995 50  0000 C CNN
+AR Path="/5BEDDDBB/5BE45706" Ref="D12"  Part="1"
+F 0 "D12" H 4142 3995 50  0000 C CNN
 F 1 "LED" H 4142 4086 50  0000 C CNN
-F 2 "" H 4150 4250 50  0001 C CNN
+F 2 "LED_SMD:LED_0603_1608Metric_Pad1.05x0.95mm_HandSolder" H 4150 4250 50  0001 C CNN
 F 3 "~" H 4150 4250 50  0001 C CNN
 	1    4150 4250
@@
 Text Label 2350 3250 0    50   ~ 0
 in[0..7]
+$Comp
+L Device:R_Pack04 RN1
+U 1 1 5BEE3417
+P 5000 3750
+F 0 "RN1" V 4583 3750 50  0000 C CNN
+F 1 "R_Pack04" V 4674 3750 50  0000 C CNN
+F 2 "Resistor_SMD:R_Array_Concave_4x0603" V 5275 3750 50  0001 C CNN
+F 3 "~" H 5000 3750 50  0001 C CNN
+	1    5000 3750
+	0    -1   1    0
+$EndComp
+$Comp
+L Device:R_Pack04 RN2
+U 1 1 5BEE3486
+P 5000 4150
+F 0 "RN2" V 4583 4150 50  0000 C CNN
+F 1 "R_Pack04" V 4674 4150 50  0000 C CNN
+F 2 "Resistor_SMD:R_Array_Concave_4x0603" V 5275 4150 50  0001 C CNN
+F 3 "~" H 5000 4150 50  0001 C CNN
+	1    5000 4150
+	0    -1   1    0
+$EndComp
+Wire Wire Line
+	5200 4250 5200 4450
+Connection ~ 5200 3650
+Connection ~ 5200 3750
+Connection ~ 5200 3850
+Connection ~ 5200 3950
+Connection ~ 5200 4250
+Connection ~ 5200 4050
+Connection ~ 5200 4150
+Wire Wire Line
+	5200 3550 5200 3650
+Wire Wire Line
+	5200 3650 5200 3750
+Wire Wire Line
+	5200 3750 5200 3850
+Wire Wire Line
+	5200 3850 5200 3950
+Wire Wire Line
+	5200 3950 5200 4050
+Wire Wire Line
+	5200 4050 5200 4150
+Wire Wire Line
+	5200 4150 5200 4250
 Wire Bus Line
 	2750 3250 2750 4150

Commit message: 8-bit-Const routed
Parts:
- RN3: renamed from RN1; footprint Resistor_SMD:R_Array_Concave_4x0603 -> Resistor_SMD:R_Array_Convex_4x0603
- RN4: renamed from RN2; footprint Resistor_SMD:R_Array_Concave_4x0603 -> Resistor_SMD:R_Array_Convex_4x0603
- renumbered D9 to D1, D10 to D2, D11 to D3, D12 to D4, D13 to D5, D14 to D6, D15 to D7, D16 to D8
Changed lines of the file:
@@
 $Descr A4 11693 8268
 encoding utf-8
-Sheet 11 12
+Sheet 11 3
 Title ""
 Date ""
@@
 AR Path="/5BE1CDAC/5BF7F814/5BE44C99" Ref="U?"  Part="1"
 AR Path="/5BE1CDAC/5BF87C71/5BE44C99" Ref="U?"  Part="1"
-AR Path="/5BEDDDBB/5BE44C99" Ref="U1"  Part="1"
+AR Path="/5BEDDDBB/5BE44C99" Ref="U?"  Part="1"
+AR Path="/5BF6FAD3/5BE44C99" Ref="U?"  Part="1"
+AR Path="/5BF7F814/5BE44C99" Ref="U?"  Part="1"
+AR Path="/5BF87C71/5BE44C99" Ref="U?"  Part="1"
+AR Path="/5BF47298/5BE44C99" Ref="U1"  Part="1"
 F 0 "U1" H 3500 4317 50  0000 C CNN
 F 1 "ULN2803A" H 3500 4226 50  0000 C CNN
@@
 $EndComp
 $Comp
-L power:GND #PWR035
+L power:GND #PWR?
 U 1 1 5BE4524F
 P 3500 4550
-F 0 "#PWR035" H 3500 4300 50  0001 C CNN
+AR Path="/5BF6FAD3/5BE4524F" Ref="#PWR?"  Part="1"
+AR Path="/5BF7F814/5BE4524F" Ref="#PWR?"  Part="1"
+AR Path="/5BF87C71/5BE4524F" Ref="#PWR?"  Part="1"
+AR Path="/5BF47298/5BE4524F" Ref="#PWR05"  Part="1"
+F 0 "#PWR05" H 3500 4300 50  0001 C CNN
 F 1 "GND" H 3505 4377 50  0000 C CNN
 F 2 "" H 3500 4550 50  0001 C CNN
@@
 $EndComp
 $Comp
-L power:+3.3V #PWR036
+L power:+3.3V #PWR?
 U 1 1 5BE4527A
 P 3950 3350
-F 0 "#PWR036" H 3950 3200 50  0001 C CNN
+AR Path="/5BF6FAD3/5BE4527A" Ref="#PWR?"  Part="1"
+AR Path="/5BF7F814/5BE4527A" Ref="#PWR?"  Part="1"
+AR Path="/5BF87C71/5BE4527A" Ref="#PWR?"  Part="1"
+AR Path="/5BF47298/5BE4527A" Ref="#PWR06"  Part="1"
+F 0 "#PWR06" H 3950 3200 50  0001 C CNN
 F 1 "+3.3V" H 3965 3523 50  0000 C CNN
 F 2 "" H 3950 3350 50  0001 C CNN
@@
 AR Path="/5BE1CDAC/5BF7F814/5BE455EA" Ref="D?"  Part="1"
 AR Path="/5BE1CDAC/5BF87C71/5BE455EA" Ref="D?"  Part="1"
-AR Path="/5BEDDDBB/5BE455EA" Ref="D13"  Part="1"
-F 0 "D13" H 4492 3295 50  0000 C CNN
+AR Path="/5BEDDDBB/5BE455EA" Ref="D?"  Part="1"
+AR Path="/5BF6FAD3/5BE455EA" Ref="D?"  Part="1"
+AR Path="/5BF7F814/5BE455EA" Ref="D?"  Part="1"
+AR Path="/5BF87C71/5BE455EA" Ref="D?"  Part="1"
+AR Path="/5BF47298/5BE455EA" Ref="D5"  Part="1"
+F 0 "D5" H 4492 3295 50  0000 C CNN
 F 1 "LED" H 4492 3386 50  0000 C CNN
 F 2 "LED_SMD:LED_0603_1608Metric_Pad1.05x0.95mm_HandSolder" H 4500 3550 50  0001 C CNN
@@
 AR Path="/5BE1CDAC/5BF7F814/5BE45642" Ref="D?"  Part="1"
 AR Path="/5BE1CDAC/5BF87C71/5BE45642" Ref="D?"  Part="1"
-AR Path="/5BEDDDBB/5BE45642" Ref="D9"  Part="1"
-F 0 "D9" H 4142 3395 50  0000 C CNN
+AR Path="/5BEDDDBB/5BE45642" Ref="D?"  Part="1"
+AR Path="/5BF6FAD3/5BE45642" Ref="D?"  Part="1"
+AR Path="/5BF7F814/5BE45642" Ref="D?"  Part="1"
+AR Path="/5BF87C71/5BE45642" Ref="D?"  Part="1"
+AR Path="/5BF47298/5BE45642" Ref="D1"  Part="1"
+F 0 "D1" H 4142 3395 50  0000 C CNN
 F 1 "LED" H 4142 3486 50  0000 C CNN
 F 2 "LED_SMD:LED_0603_1608Metric_Pad1.05x0.95mm_HandSolder" H 4150 3650 50  0001 C CNN
@@
 AR Path="/5BE1CDAC/5BF7F814/5BE45666" Ref="D?"  Part="1"
 AR Path="/5BE1CDAC/5BF87C71/5BE45666" Ref="D?"  Part="1"
-AR Path="/5BEDDDBB/5BE45666" Ref="D14"  Part="1"
-F 0 "D14" H 4492 3495 50  0000 C CNN
+AR Path="/5BEDDDBB/5BE45666" Ref="D?"  Part="1"
+AR Path="/5BF6FAD3/5BE45666" Ref="D?"  Part="1"
+AR Path="/5BF7F814/5BE45666" Ref="D?"  Part="1"
+AR Path="/5BF87C71/5BE45666" Ref="D?"  Part="1"
+AR Path="/5BF47298/5BE45666" Ref="D6"  Part="1"
+F 0 "D6" H 4492 3495 50  0000 C CNN
 F 1 "LED" H 4492 3586 50  0000 C CNN
 F 2 "LED_SMD:LED_0603_1608Metric_Pad1.05x0.95mm_HandSolder" H 4500 3750 50  0001 C CNN
@@
 AR Path="/5BE1CDAC/5BF7F814/5BE45682" Ref="D?"  Part="1"
 AR Path="/5BE1CDAC/5BF87C71/5BE45682" Ref="D?"  Part="1"
-AR Path="/5BEDDDBB/5BE45682" Ref="D10"  Part="1"
-F 0 "D10" H 4142 3595 50  0000 C CNN
+AR Path="/5BEDDDBB/5BE45682" Ref="D?"  Part="1"
+AR Path="/5BF6FAD3/5BE45682" Ref="D?"  Part="1"
+AR Path="/5BF7F814/5BE45682" Ref="D?"  Part="1"
+AR Path="/5BF87C71/5BE45682" Ref="D?"  Part="1"
+AR Path="/5BF47298/5BE45682" Ref="D2"  Part="1"
+F 0 "D2" H 4142 3595 50  0000 C CNN
 F 1 "LED" H 4142 3686 50  0000 C CNN
 F 2 "LED_SMD:LED_0603_1608Metric_Pad1.05x0.95mm_HandSolder" H 4150 3850 50  0001 C CNN
@@
 AR Path="/5BE1CDAC/5BF7F814/5BE456A0" Ref="D?"  Part="1"
 AR Path="/5BE1CDAC/5BF87C71/5BE456A0" Ref="D?"  Part="1"
-AR Path="/5BEDDDBB/5BE456A0" Ref="D15"  Part="1"
-F 0 "D15" H 4492 3695 50  0000 C CNN
+AR Path="/5BEDDDBB/5BE456A0" Ref="D?"  Part="1"
+AR Path="/5BF6FAD3/5BE456A0" Ref="D?"  Part="1"
+AR Path="/5BF7F814/5BE456A0" Ref="D?"  Part="1"
+AR Path="/5BF87C71/5BE456A0" Ref="D?"  Part="1"
+AR Path="/5BF47298/5BE456A0" Ref="D7"  Part="1"
+F 0 "D7" H 4492 3695 50  0000 C CNN
 F 1 "LED" H 4492 3786 50  0000 C CNN
 F 2 "LED_SMD:LED_0603_1608Metric_Pad1.05x0.95mm_HandSolder" H 4500 3950 50  0001 C CNN
@@
 AR Path="/5BE1CDAC/5BF7F814/5BE456C0" Ref="D?"  Part="1"
 AR Path="/5BE1CDAC/5BF87C71/5BE456C0" Ref="D?"  Part="1"
-AR Path="/5BEDDDBB/5BE456C0" Ref="D11"  Part="1"
-F 0 "D11" H 4142 3795 50  0000 C CNN
+AR Path="/5BEDDDBB/5BE456C0" Ref="D?"  Part="1"
+AR Path="/5BF6FAD3/5BE456C0" Ref="D?"  Part="1"
+AR Path="/5BF7F814/5BE456C0" Ref="D?"  Part="1"
+AR Path="/5BF87C71/5BE456C0" Ref="D?"  Part="1"
+AR Path="/5BF47298/5BE456C0" Ref="D3"  Part="1"
+F 0 "D3" H 4142 3795 50  0000 C CNN
 F 1 "LED" H 4142 3886 50  0000 C CNN
 F 2 "LED_SMD:LED_0603_1608Metric_Pad1.05x0.95mm_HandSolder" H 4150 4050 50  0001 C CNN
@@
 AR Path="/5BE1CDAC/5BF7F814/5BE456E2" Ref="D?"  Part="1"
 AR Path="/5BE1CDAC/5BF87C71/5BE456E2" Ref="D?"  Part="1"
-AR Path="/5BEDDDBB/5BE456E2" Ref="D16"  Part="1"
-F 0 "D16" H 4492 3895 50  0000 C CNN
+AR Path="/5BEDDDBB/5BE456E2" Ref="D?"  Part="1"
+AR Path="/5BF6FAD3/5BE456E2" Ref="D?"  Part="1"
+AR Path="/5BF7F814/5BE456E2" Ref="D?"  Part="1"
+AR Path="/5BF87C71/5BE456E2" Ref="D?"  Part="1"
+AR Path="/5BF47298/5BE456E2" Ref="D8"  Part="1"
+F 0 "D8" H 4492 3895 50  0000 C CNN
 F 1 "LED" H 4492 3986 50  0000 C CNN
 F 2 "LED_SMD:LED_0603_1608Metric_Pad1.05x0.95mm_HandSolder" H 4500 4150 50  0001 C CNN
@@
 AR Path="/5BE1CDAC/5BF7F814/5BE45706" Ref="D?"  Part="1"
 AR Path="/5BE1CDAC/5BF87C71/5BE45706" Ref="D?"  Part="1"
-AR Path="/5BEDDDBB/5BE45706" Ref="D12"  Part="1"
-F 0 "D12" H 4142 3995 50  0000 C CNN
+AR Path="/5BEDDDBB/5BE45706" Ref="D?"  Part="1"
+AR Path="/5BF6FAD3/5BE45706" Ref="D?"  Part="1"
+AR Path="/5BF7F814/5BE45706" Ref="D?"  Part="1"
+AR Path="/5BF87C71/5BE45706" Ref="D?"  Part="1"
+AR Path="/5BF47298/5BE45706" Ref="D4"  Part="1"
+F 0 "D4" H 4142 3995 50  0000 C CNN
 F 1 "LED" H 4142 4086 50  0000 C CNN
 F 2 "LED_SMD:LED_0603_1608Metric_Pad1.05x0.95mm_HandSolder" H 4150 4250 50  0001 C CNN
@@
 in[0..7]
 $Comp
-L Device:R_Pack04 RN1
+L Device:R_Pack04 RN?
 U 1 1 5BEE3417
-P 5000 3750
-F 0 "RN1" V 4583 3750 50  0000 C CNN
-F 1 "R_Pack04" V 4674 3750 50  0000 C CNN
-F 2 "Resistor_SMD:R_Array_Concave_4x0603" V 5275 3750 50  0001 C CNN
-F 3 "~" H 5000 3750 50  0001 C CNN
-	1    5000 3750
-	0    -1   1    0
-$EndComp
-$Comp
-L Device:R_Pack04 RN2
+P 5000 3650
+AR Path="/5BF6FAD3/5BEE3417" Ref="RN?"  Part="1"
+AR Path="/5BF7F814/5BEE3417" Ref="RN?"  Part="1"
+AR Path="/5BF87C71/5BEE3417" Ref="RN?"  Part="1"
+AR Path="/5BF47298/5BEE3417" Ref="RN3"  Part="1"
+F 0 "RN3" V 4583 3650 50  0000 C CNN
+F 1 "R_Pack04" V 4674 3650 50  0000 C CNN
+F 2 "Resistor_SMD:R_Array_Convex_4x0603" V 5275 3650 50  0001 C CNN
+F 3 "~" H 5000 3650 50  0001 C CNN
+	1    5000 3650
+	0    1    -1   0
+$EndComp
+$Comp
+L Device:R_Pack04 RN?
 U 1 1 5BEE3486
-P 5000 4150
-F 0 "RN2" V 4583 4150 50  0000 C CNN
-F 1 "R_Pack04" V 4674 4150 50  0000 C CNN
-F 2 "Resistor_SMD:R_Array_Concave_4x0603" V 5275 4150 50  0001 C CNN
-F 3 "~" H 5000 4150 50  0001 C CNN
-	1    5000 4150
-	0    -1   1    0
-$EndComp
-Wire Wire Line
-	5200 4250 5200 4450
-Connection ~ 5200 3650
-Connection ~ 5200 3750
-Connection ~ 5200 3850
-Connection ~ 5200 3950
-Connection ~ 5200 4250
-Connection ~ 5200 4050
-Connection ~ 5200 4150
+P 5000 4050
+AR Path="/5BF6FAD3/5BEE3486" Ref="RN?"  Part="1"
+AR Path="/5BF7F814/5BEE3486" Ref="RN?"  Part="1"
+AR Path="/5BF87C71/5BEE3486" Ref="RN?"  Part="1"
+AR Path="/5BF47298/5BEE3486" Ref="RN4"  Part="1"
+F 0 "RN4" V 4583 4050 50  0000 C CNN
+F 1 "R_Pack04" V 4674 4050 50  0000 C CNN
+F 2 "Resistor_SMD:R_Array_Convex_4x0603" V 5275 4050 50  0001 C CNN
+F 3 "~" H 5000 4050 50  0001 C CNN
+	1    5000 4050
+	0    1    -1   0
+$EndComp
 Wire Wire Line
 	5200 3550 5200 3650
-Wire Wire Line
-	5200 3650 5200 3750
-Wire Wire Line
-	5200 3750 5200 3850
-Wire Wire Line
-	5200 3850 5200 3950
-Wire Wire Line
-	5200 3950 5200 4050
-Wire Wire Line
-	5200 4050 5200 4150
-Wire Wire Line
-	5200 4150 5200 4250
 Wire Bus Line
 	2750 3250 2750 4150
+Connection ~ 5200 3650
+Wire Wire Line
+	5200 3650 5200 3750
+Connection ~ 5200 3750
+Wire Wire Line
+	5200 3750 5200 3850
+Connection ~ 5200 3850
+Wire Wire Line
+	5200 3850 5200 3950
+Connection ~ 5200 3950
+Wire Wire Line
+	5200 3950 5200 4050
+Connection ~ 5200 4050
+Wire Wire Line
+	5200 4050 5200 4150
+Connection ~ 5200 4150
+Wire Wire Line
+	5200 4150 5200 4250
+Connection ~ 5200 4250
+Wire Wire Line
+	5200 4250 5200 4450
 $EndSCHEMATC
