File: 8-BitSteck/MUX.sch (KiCad schematic (older format))
At the start: 4 parts

Commit message: Add files via upload
Connections:
- net labels added: A[0..7], B[0..7], OUT[0..7], S, a0, a1, a2, a3, a4, a5, a6, a7, a[0..7], b0, b1, b2, b3, b4, b5, b6, b7, b[0..7], out0, out1, out2, out3, out4, out5, out6, out7, out[0..7], ~E
- wire segments 92 -> 98

Commit message: 8-bit-Const routed
Parts:
- R1, R2: renamed from R?; footprint (none) -> Resistor_SMD:R_0603_1608Metric_Pad1.05x0.95mm_HandSolder
- U1, U2: renamed from U?; footprint (none) -> Package_SO:SOIC-16_3.9x9.9mm_P1.27mm
Connections:
- wire segments 98 -> 99
Changed lines of the file:
@@
 EESchema Schematic File Version 4
-LIBS:8-BitSteck-cache
 EELAYER 26 0
 EELAYER END
 $Descr A4 11693 8268
 encoding utf-8
-Sheet 35 66
+Sheet 1 9
 Title ""
 Date ""
@@
 $EndDescr
 $Comp
-L 74xx:74LS157 U?
+L 74xx:74LS157 U1
 U 1 1 5BE1CE32
 P 5850 2100
-F 0 "U?" H 5850 3178 50  0000 C CNN
+F 0 "U1" H 5850 3178 50  0000 C CNN
 F 1 "74LS157" H 5850 3087 50  0000 C CNN
-F 2 "" H 5850 2100 50  0001 C CNN
+F 2 "Package_SO:SOIC-16_3.9x9.9mm_P1.27mm" H 5850 2100 50  0001 C CNN
 F 3 "http://www.ti.com/lit/gpn/sn74LS157" H 5850 2100 50  0001 C CNN
 	1    5850 2100
@@
 $EndComp
 $Comp
-L 74xx:74LS157 U?
+L 74xx:74LS157 U2
 U 1 1 5BE1CE9B
 P 5850 4900
-F 0 "U?" H 5850 5978 50  0000 C CNN
+F 0 "U2" H 5850 5978 50  0000 C CNN
 F 1 "74LS157" H 5850 5887 50  0000 C CNN
-F 2 "" H 5850 4900 50  0001 C CNN
+F 2 "Package_SO:SOIC-16_3.9x9.9mm_P1.27mm" H 5850 4900 50  0001 C CNN
 F 3 "http://www.ti.com/lit/gpn/sn74LS157" H 5850 4900 50  0001 C CNN
 	1    5850 4900
@@
 $EndComp
 $Comp
-L power:GND #PWR?
+L power:GND #PWR04
 U 1 1 5BE1D033
 P 5850 6050
-F 0 "#PWR?" H 5850 5800 50  0001 C CNN
+F 0 "#PWR04" H 5850 5800 50  0001 C CNN
 F 1 "GND" H 5855 5877 50  0000 C CNN
 F 2 "" H 5850 6050 50  0001 C CNN
@@
 $EndComp
 $Comp
-L power:GND #PWR?
+L power:GND #PWR02
 U 1 1 5BE1D059
 P 5850 3250
-F 0 "#PWR?" H 5850 3000 50  0001 C CNN
+F 0 "#PWR02" H 5850 3000 50  0001 C CNN
 F 1 "GND" H 5855 3077 50  0000 C CNN
 F 2 "" H 5850 3250 50  0001 C CNN
@@
 AR Path="/5BD2B43F/5BE1D189" Ref="R?"  Part="1"
 AR Path="/5BE1CDAC/5BE1D189" Ref="R?"  Part="1"
-F 0 "R?" H 5420 5846 50  0000 L CNN
+AR Path="/5BE1D189" Ref="R2"  Part="1"
+F 0 "R2" H 5420 5846 50  0000 L CNN
 F 1 "R_default" H 5420 5755 50  0000 L CNN
-F 2 "" V 5280 5800 50  0001 C CNN
+F 2 "Resistor_SMD:R_0603_1608Metric_Pad1.05x0.95mm_HandSolder" V 5280 5800 50  0001 C CNN
 F 3 "~" H 5350 5800 50  0001 C CNN
 	1    5350 5800
@@
 L Device:R R?
 U 1 1 5BE1D1AA
-P 5350 3000
+P 5250 3000
 AR Path="/5BD2B43F/5BE1D1AA" Ref="R?"  Part="1"
 AR Path="/5BE1CDAC/5BE1D1AA" Ref="R?"  Part="1"
-F 0 "R?" H 5420 3046 50  0000 L CNN
-F 1 "R_default" H 5420 2955 50  0000 L CNN
-F 2 "" V 5280 3000 50  0001 C CNN
-F 3 "~" H 5350 3000 50  0001 C CNN
-	1    5350 3000
-	1    0    0    -1
-$EndComp
-Wire Wire Line
-	5350 2800 5350 2850
-Wire Wire Line
-	5350 3150 5850 3150
+AR Path="/5BE1D1AA" Ref="R1"  Part="1"
+F 0 "R1" H 5320 3046 50  0000 L CNN
+F 1 "R_default" H 5320 2955 50  0000 L CNN
+F 2 "Resistor_SMD:R_0603_1608Metric_Pad1.05x0.95mm_HandSolder" V 5180 3000 50  0001 C CNN
+F 3 "~" H 5250 3000 50  0001 C CNN
+	1    5250 3000
+	1    0    0    -1
+$EndComp
 Connection ~ 5850 3150
 Wire Wire Line
@@
 	5350 5650 5350 5600
 $Comp
-L power:+3.3V #PWR?
+L power:+3.3V #PWR01
 U 1 1 5BE1D47B
 P 5850 1150
-F 0 "#PWR?" H 5850 1000 50  0001 C CNN
+F 0 "#PWR01" H 5850 1000 50  0001 C CNN
 F 1 "+3.3V" H 5865 1323 50  0000 C CNN
 F 2 "" H 5850 1150 50  0001 C CNN
@@
 $EndComp
 $Comp
-L power:+3.3V #PWR?
+L power:+3.3V #PWR03
 U 1 1 5BE1D4F2
 P 5850 3950
-F 0 "#PWR?" H 5850 3800 50  0001 C CNN
+F 0 "#PWR03" H 5850 3800 50  0001 C CNN
 F 1 "+3.3V" H 5865 4123 50  0000 C CNN
 F 2 "" H 5850 3950 50  0001 C CNN
@@
 	4500 5300 5350 5300
 Wire Wire Line
-	5350 2700 5150 2700
+	5350 2700 5250 2700
 Wire Wire Line
 	5150 2700 5150 5500
@@
 Wire Wire Line
 	5050 5600 4050 5600
-Connection ~ 5350 2800
 Entry Wire Line
 	3550 2300 3650 2400
@@
 Wire Wire Line
 	3750 5850 4050 5850
+Wire Wire Line
+	5250 3150 5850 3150
+Wire Wire Line
+	5250 2850 5250 2700
+Wire Bus Line
+	3550 4100 3550 4250
+Wire Bus Line
+	3550 2850 3550 3000
+Wire Bus Line
+	3550 3350 3550 3650
+Wire Bus Line
+	3550 2100 3550 2400
+Wire Bus Line
+	8250 3800 8250 3950
 Wire Bus Line
 	8250 3100 8250 3350
 Wire Bus Line
-	8250 3800 8250 3950
-Wire Bus Line
-	3550 2100 3550 2400
-Wire Bus Line
-	3550 3350 3550 3650
-Wire Bus Line
-	3550 2850 3550 3000
-Wire Bus Line
-	3550 4100 3550 4250
+	3550 3650 3550 4100
+Wire Bus Line
+	3550 2400 3550 2850
 Wire Bus Line
 	8250 3350 8250 3800
-Wire Bus Line
-	3550 2400 3550 2850
-Wire Bus Line
-	3550 3650 3550 4100
+Connection ~ 5250 2700
+Wire Wire Line
+	5250 2700 5150 2700
 $EndSCHEMATC
